File: docs/Schematics/Driver/Driver.kicad_pcb (KiCad board)
At the start: 4 copper layers, 115.7 x 107 mm, 61 parts, among them J1 AUX_IOref, J10 AUX_3V3, J11 AUX_GND, J12 PH_MC, J13 A1363xKTTN-1_front_left, J14 A1363xKTTN-1_midle_left, J15 A1363xKTTN-1_rear_left, J16 A1363xKTTN-1_front_right, J17 PH_MC, J18 A1363xKTTN-1_midle_right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

Commit message: Changed a few nets to make the routing posible
Parts:
- moved R10 27.1 mm to (153.3, 152.9), turned to 90 degrees
- moved R11 22.9 mm to (130.1, 137.6)
- moved R1 20.4 mm to (185.1, 56.1), turned to -90 degrees
- moved R4 19.7 mm to (205.5, 71.3), turned to 90 degrees
- moved R2 19.5 mm to (191.9, 71.3), turned to 90 degrees
- moved R3 19.2 mm to (198.7, 56.1), turned to -90 degrees
- moved R5 17.6 mm to (207.7, 137.5), turned to -90 degrees
- moved R12 16.4 mm to (137.8, 152.9), turned to 90 degrees
- moved R7 15.8 mm to (185.4, 137.5), turned to -90 degrees
- moved R9 7.67 mm to (145.6, 137.6)
- moved R6 7.10 mm to (200.2, 152.8)
- moved J16 5.86 mm to (226.5, 145.0)
- moved J18 4.36 mm to (226.5, 130.2)
- moved J19 2.94 mm to (226.5, 115.4)
- moved J13 2.81 mm to (226.5, 71.0)
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Connections:
- J2 pad 6: /MWL/CS -> /MMR/CS
- J2 pad 8: /MMR/CS -> /MWL/CS
- J6 pad 10: /MRL/INB -> /MRR/INB
- J6 pad 12: /MRL/PWM -> /MRR/PWM
- J6 pad 14: /MRR/PWM -> /MRL/PWM
- J6 pad 16: /MRR/INB -> /MRL/INB
- J6 pad 18: /MR/INA -> /MRL/INA
- J6 pad 20: /MRR/EN -> /MRL/EN
- J6 pad 6: /MRL/EN -> /MRR/EN
- J6 pad 8: /MRL/INA -> /MR/INA
- J7 pad 10: /MMR/PWM -> /MML/PWM
- J7 pad 12: /MMR/INB -> /MML/INB
- J7 pad 14: /MMR/INA -> /MML/INA
- J7 pad 16: /MMR/EN -> /MML/EN
- J7 pad 2: /MML/EN -> /MMR/EN
- J7 pad 4: /MML/INA -> /MMR/INA
- J7 pad 6: /MML/INB -> /MMR/INB
- J7 pad 8: /MML/PWM -> /MMR/PWM
Routing:
- net /MFL/CS: track 0.00 -> 131.5 mm, vias 0 -> 1
- net /MFR/CS: track 0.00 -> 109.2 mm, vias 0 -> 1
- net /Motor Driver Front/Dual_VNH3SP30/2DIAG/EN: track 0.00 -> 100.9 mm
- net /Motor Driver Front/Dual_VNH3SP30/2INA: track 0.00 -> 92.9 mm, vias 0 -> 1
- net /MRR/CS: track 0.00 -> 64.4 mm
- net /MML/INB: track 0.00 -> 54.5 mm
- net /MML/PWM: track 0.00 -> 53.6 mm
- net /MRL/CS: track 0.00 -> 51.4 mm
- net /MML/INA: track 0.00 -> 45.8 mm
- net /MML/EN: track 0.00 -> 43.8 mm
- net /MWL/CS: track 0.00 -> 42.9 mm
- net /MR/INA: track 0.00 -> 36.6 mm
- net /MRR/EN: track 0.00 -> 35.5 mm
- net /MMR/CS: track 0.00 -> 33.4 mm
- net /MRR/PWM: track 0.00 -> 29.2 mm
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Other:
- board size 115.7 x 107 mm -> 116 x 107 mm
