File: docs/Schematics/Driver/ArtyZ7.kicad_sch (KiCad schematic)
At the start: 7 parts, among them J1 Conn_01x02_Female, J2 Conn_02x06_Counter_Clockwise, J4 PH_PWR, J5 Conn_01x06_Female, J6 PH_IO1, J7 PH_IO2, J8 Conn_01x04_Female

Commit message: Started routing the pcb.
Parts:
- J1: value Conn_01x02_Female -> AUX_IOref
- J2: value Conn_02x06_Counter_Clockwise -> PH_Ain
- J4, J7: footprint Connector_PinHeader_2.54mm:PinHeader_2x16_P2.54mm_Vertical -> Connector_PinHeader_2.54mm:PinHeader_2x08_P2.54mm_Vertical
- J5: value Conn_01x06_Female -> AUX_AIO
- J6: footprint Connector_PinHeader_2.54mm:PinHeader_2x20_P2.54mm_Vertical -> Connector_PinHeader_2.54mm:PinHeader_2x10_P2.54mm_Vertical
- J8: value Conn_01x04_Female -> AUX_Ain
Connections:
- net +3.3V: now also J4.8 (Pin_8); no longer J4.7 (Pin_7)
- net +5V: now also J4.10 (Pin_10); no longer J4.9 (Pin_9)
- net A0: now also J2.2 (Pin_2); no longer J2.1 (Pin_1)
- net A1: now also J2.4 (Pin_4); no longer J2.3 (Pin_3)
- net A2: now also J2.6 (Pin_6); no longer J2.5 (Pin_5)
- net A3: now also J2.8 (Pin_8); no longer J2.7 (Pin_7)
- net A4: now also J2.10 (Pin_10); no longer J2.9 (Pin_9)
- net A5: now also J2.12 (Pin_12); no longer J2.11 (Pin_11)
- net GNDD: now also J4.12 (Pin_12), J6.7 (Pin_7); no longer J4.11 (Pin_11), J6.8 (Pin_8)
- net IO0: now also J7.15 (Pin_15); no longer J7.16 (Pin_16)
- net IO1: now also J7.13 (Pin_13); no longer J7.14 (Pin_14)
- net IO10: now also J6.15 (Pin_15); no longer J6.16 (Pin_16)
- net IO11: now also J6.13 (Pin_13); no longer J6.14 (Pin_14)
- net IO12: now also J6.11 (Pin_11); no longer J6.12 (Pin_12)
- net IO13: now also J6.9 (Pin_9); no longer J6.10 (Pin_10)
- net IO2: now also J7.11 (Pin_11); no longer J7.12 (Pin_12)
- net IO26: now also J7.16 (Pin_16); no longer J7.15 (Pin_15)
- net IO27: now also J7.14 (Pin_14); no longer J7.13 (Pin_13)
- net IO28: now also J7.12 (Pin_12); no longer J7.11 (Pin_11)
- net IO29: now also J7.10 (Pin_10); no longer J7.9 (Pin_9)
- net IO3: now also J7.9 (Pin_9); no longer J7.10 (Pin_10)
- net IO30: now also J7.8 (Pin_8); no longer J7.7 (Pin_7)
- net IO31: now also J7.6 (Pin_6); no longer J7.5 (Pin_5)
- net IO32: now also J7.4 (Pin_4); no longer J7.3 (Pin_3)
- net IO33: now also J7.2 (Pin_2); no longer J7.1 (Pin_1)
- net IO34: now also J6.20 (Pin_20); no longer J6.19 (Pin_19)
- net IO35: now also J6.18 (Pin_18); no longer J6.17 (Pin_17)
- net IO36: now also J6.16 (Pin_16); no longer J6.15 (Pin_15)
- net IO37: now also J6.14 (Pin_14); no longer J6.13 (Pin_13)
- net IO38: now also J6.12 (Pin_12); no longer J6.11 (Pin_11)
- net IO39: now also J6.10 (Pin_10); no longer J6.9 (Pin_9)
- net IO4: now also J7.7 (Pin_7); no longer J7.8 (Pin_8)
- net IO40: now also J6.8 (Pin_8); no longer J6.7 (Pin_7)
- net IO41: now also J6.6 (Pin_6); no longer J6.5 (Pin_5)
- net IO42: now also J6.5 (Pin_5); no longer J6.6 (Pin_6)
- net IO5: now also J7.5 (Pin_5); no longer J7.6 (Pin_6)
- net IO6: now also J7.3 (Pin_3); no longer J7.4 (Pin_4)
- net IO7: now also J7.1 (Pin_1); no longer J7.2 (Pin_2)
- net IO8: now also J6.19 (Pin_19); no longer J6.20 (Pin_20)
- net IO9: now also J6.17 (Pin_17); no longer J6.18 (Pin_18)
- net IOREF: now also J4.4 (Pin_4); no longer J4.3 (Pin_3)
- net RST: now also J4.6 (Pin_6); no longer J4.5 (Pin_5)
- net SCL: now also J6.1 (Pin_1); no longer J6.2 (Pin_2)
- net SDA: now also J6.3 (Pin_3); no longer J6.4 (Pin_4)
- net XVREF: now also J4.15 (Pin_15); no longer J4.16 (Pin_16)
- net v_n: now also J4.11 (Pin_11); no longer J4.12 (Pin_12)
- net v_p: now also J4.9 (Pin_9); no longer J4.10 (Pin_10)
- net at J5.1 (Pin_1): now also J2.1 (Pin_1); no longer J2.2 (Pin_2)
- net at J5.2 (Pin_2): now also J2.3 (Pin_3); no longer J2.4 (Pin_4)
- net at J5.3 (Pin_3): now also J2.5 (Pin_5); no longer J2.6 (Pin_6)
- net at J5.4 (Pin_4): now also J2.7 (Pin_7); no longer J2.8 (Pin_8)
- net at J5.5 (Pin_5): now also J2.9 (Pin_9); no longer J2.10 (Pin_10)
- net at J5.6 (Pin_6): now also J2.11 (Pin_11); no longer J2.12 (Pin_12)
Other:
- note added: "CUT"
- note removed: "No entry in card"

Commit message: First version of the routed board is done
Other:
- title: Arty Z7 IO expander card -> Arty Z7 IO Board
Changed lines of the file:
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@@
   (paper "A4")
   (title_block
-    (title "Arty Z7 IO expander card")
+    (title "Arty Z7 IO Board")
     (date "2022-12-24")
-    (rev "0.1")
+    (rev "${VER}")
     (company "HiQ")
   )
