Commit message: Add mesh model to urdf

File: ndo_description/urdf/ndo.urdf (robot description, URDF)
Before this commit: robot ndo, 2 links, 1 joints
Links:
- link base_link: geometry visual mesh filename=package://ndo_description/mesh/base.stl
Joints:
- joint base_joint: origin xyz=0.0 0.0 ${-(wheel_radius+wheel_zoff)} rpy=0 0 0 -> xyz=0.0 0.0 ${footprint_zoff} rpy=0 0 0
