Commit message: Refactor urdf

File: ndo_description/urdf/controller.xacro (robot description, xacro)
@@ -20,4 +20,11 @@
     <xacro:if value="$(arg use_sim_ctrl)">
         <!-- Gazebo simulation controller -->
+        <gazebo>
+            <plugin filename="libgazebo_ros2_control.so" name="gazebo_ros2_control">
+                <robot_param>robot_description</robot_param>
+                <robot_param_node>robot_state_publisher</robot_param_node>
+                <parameters>$(find ndo_controller)/config/controllers.yaml</parameters>
+            </plugin>
+        </gazebo>
         <ros2_control name="GazeboSystem" type="system">
             <hardware>

File: ndo_description/urdf/ndo.urdf.xacro (robot description, xacro)
@@ -1,8 +1,6 @@
 <robot xmlns:xacro="http://www.ros.org/wiki/xacro" name="ndo">
-    <!-- Include parts -->
+    <!-- Include macros -->
     <xacro:include filename="$(find ndo_description)/urdf/wheel.urdf.xacro"/>
-    <!-- Include dynamics/controller/materials -->
-    <xacro:include filename="$(find ndo_description)/urdf/materials.gazebo.xacro"/>
-    <xacro:include filename="$(find ndo_description)/urdf/ndo.gazebo.xacro"/>
+    <!-- Include controller -->
     <xacro:include filename="$(find ndo_description)/urdf/controller.xacro"/>
     <!-- Base properties -->
@@ -11,5 +9,7 @@
     <xacro:property name="base_height" value="0.072"/>
     <xacro:property name="footprint_zoff" value="${(0.135-base_height/2)}"/>
-    <xacro:property name="caster_xoff" value="0.14"/>
+    <!-- Spring properties -->
+    <xacro:property name="spring_stiffness" value="4"/>
+    <!-- Links and joints! -->
     <link name="base_link"/>
     <link name="body_link">
@@ -35,5 +35,10 @@
         </inertial>
     </link>
-    <!-- Base footprint of the robot which is the center reference -->
+    <!-- Base footprint of the robot which is the center reference. This should
+         probably be dynamic since the robot has a suspension system. You
+         always want the base_footprint to be at ground level to represent
+         the 2D view and that is not true if the footprint follows the suspension
+         "bouncing" of the robot. -->
+    <!-- TODO Should probably be dynamic since the robot has a suspension system -->
     <link name="base_footprint"/>
     <!-- Joint base_link with base_footprint to place it at ground level -->
@@ -48,9 +53,13 @@
         <origin xyz="0 0 0" rpy="0 0 0"/>
     </joint>
-    <xacro:wheel position="front" side="l"/>
-    <xacro:wheel position="front" side="r"/>
-    <xacro:wheel position="middle" side="l"/>
-    <xacro:wheel position="middle" side="r"/>
-    <xacro:wheel position="back" side="l"/>
-    <xacro:wheel position="back" side="r"/>
+    <!-- Create wheels -->
+    <xacro:wheel position="front" side="l" spring_stiffness="${spring_stiffness}" spring_reference="0"/>
+    <xacro:wheel position="front" side="r" spring_stiffness="${spring_stiffness}" spring_reference="0"/>
+    <xacro:wheel position="middle" side="l" spring_stiffness="${spring_stiffness}" spring_reference="0"/>
+    <xacro:wheel position="middle" side="r" spring_stiffness="${spring_stiffness}" spring_reference="0"/>
+    <xacro:wheel position="back" side="l" spring_stiffness="${spring_stiffness}" spring_reference="0"/>
+    <xacro:wheel position="back" side="r" spring_stiffness="${spring_stiffness}" spring_reference="0"/>
+    <gazebo reference="body_link">
+        <material>Gazebo/Turquoise</material>
+    </gazebo>
 </robot>

File: ndo_description/urdf/wheel.urdf.xacro (robot description, xacro)
@@ -1,4 +1,4 @@
 <robot xmlns:xacro="http://www.ros.org/wiki/xacro" name="ndo_wheel">
-    <xacro:macro name="wheel" params="position side">
+    <xacro:macro name="wheel" params="position side spring_stiffness spring_reference">
         <xacro:property name="wheel_radius" value="0.063"/>
         <xacro:property name="wheel_width" value="0.06"/>
@@ -91,6 +91,9 @@
             <minDepth>0.005</minDepth>
         </gazebo>
-        <gazebo reference="${prefix}_adptr_link">
+        <gazebo reference="${prefix}_adptr_joint">
             <material>Gazebo/DarkYellow</material>
+            <implicitSpringDamper>true</implicitSpringDamper>
+            <springStiffness>${spring_stiffness}</springStiffness>
+            <springReference>${spring_reference}</springReference>
         </gazebo>
     </xacro:macro>
