Commit message: Add dummy link to enable inertia for the body

File: ndo_description/urdf/ndo.urdf.xacro (robot description, xacro)
@@ -12,5 +12,6 @@
     <xacro:property name="footprint_zoff" value="${(0.135-base_height/2)}"/>
     <xacro:property name="caster_xoff" value="0.14"/>
-    <link name="base_link">
+    <link name="base_link"/>
+    <link name="body_link">
         <visual>
             <geometry>
@@ -41,4 +42,9 @@
         <origin xyz="0.0 0.0 ${-footprint_zoff}" rpy="0 0 0"/>
     </joint>
+    <joint name="body_link" type="fixed">
+        <parent link="base_link"/>
+        <child link="body_link"/>
+        <origin xyz="0 0 0" rpy="0 0 0"/>
+    </joint>
     <xacro:wheel position="front" side="l"/>
     <xacro:wheel position="front" side="r"/>

Commit message: Update mesh and inertia

File: ndo_description/urdf/ndo.urdf.xacro (robot description, xacro)
@@ -31,5 +31,6 @@
             <origin xyz="-0.00275 0 0" rpy="0 0 0"/>
             <mass value="2.5"/>
-            <inertia izz="0.014021" ixy="0.0" ixz="0.0" iyy="0.012708" iyz="0.0" ixx="0.0046875"/>
+            <!-- Calculated inertia assumes that the body is a Cuboid -->
+            <inertia izz="0.031163" ixy="0.0" ixz="0.0" iyy="0.00408" iyz="0.0" ixx="0.033083"/>
         </inertial>
     </link>

File: ndo_description/urdf/wheel.urdf.xacro (robot description, xacro)
@@ -40,5 +40,5 @@
                 <origin xyz="0 0 0" rpy="0 0 0"/>
                 <mass value="0.2"/>
-                <inertia ixx="0.00024" ixy="0" ixz="0" iyy="0.00036" iyz="0" izz="0.00024"/>
+                <inertia ixx="8.4842761417e-05" ixy="-3.5206662807e-09" ixz="-8.7257106991e-09" iyy="1.2329460329e-04" iyz="5.1535165447e-09" izz="6.9099655771e-05"/>
             </inertial>
         </link>

Commit message: Reorder links base_footprint -> base_link

File: ndo_description/urdf/ndo.urdf.xacro (robot description, xacro)
@@ -39,7 +39,7 @@
     <!-- Joint base_link with base_footprint to place it at ground level -->
     <joint name="base_joint" type="fixed">
-        <parent link="base_link"/>
-        <child link="base_footprint"/>
-        <origin xyz="0.0 0.0 ${-footprint_zoff}" rpy="0 0 0"/>
+        <parent link="base_footprint"/>
+        <child link="base_link"/>
+        <origin xyz="0.0 0.0 ${footprint_zoff}" rpy="0 0 0"/>
     </joint>
     <joint name="body_link" type="fixed">

Commit message: Refactor to ndo_gazebo

File: ndo_description/urdf/ndo.urdf.xacro (robot description, xacro)
@@ -1,7 +1,10 @@
 <robot xmlns:xacro="http://www.ros.org/wiki/xacro" name="ndo">
+    <xacro:arg name="use_sim_ctrl" default="false"/>
     <!-- Include macros -->
     <xacro:include filename="$(find ndo_description)/urdf/wheel.urdf.xacro"/>
     <!-- Include controller -->
-    <xacro:include filename="$(find ndo_description)/urdf/controller.xacro"/>
+    <xacro:unless value="$(arg use_sim_ctrl)">
+        <xacro:include filename="$(find ndo_description)/urdf/diff_drive.xacro"/>
+    </xacro:unless>
     <!-- Base properties -->
     <xacro:property name="base_width" value="0.12"/>
@@ -54,12 +57,9 @@
     </joint>
     <!-- Create wheels -->
-    <xacro:wheel position="front" side="l" spring_stiffness="${spring_stiffness}" spring_reference="0"/>
-    <xacro:wheel position="front" side="r" spring_stiffness="${spring_stiffness}" spring_reference="0"/>
-    <xacro:wheel position="middle" side="l" spring_stiffness="${spring_stiffness}" spring_reference="0"/>
-    <xacro:wheel position="middle" side="r" spring_stiffness="${spring_stiffness}" spring_reference="0"/>
-    <xacro:wheel position="back" side="l" spring_stiffness="${spring_stiffness}" spring_reference="0"/>
-    <xacro:wheel position="back" side="r" spring_stiffness="${spring_stiffness}" spring_reference="0"/>
-    <gazebo reference="body_link">
-        <material>Gazebo/Turquoise</material>
-    </gazebo>
+    <xacro:wheel position="front" side="l"/>
+    <xacro:wheel position="front" side="r"/>
+    <xacro:wheel position="middle" side="l"/>
+    <xacro:wheel position="middle" side="r"/>
+    <xacro:wheel position="back" side="l"/>
+    <xacro:wheel position="back" side="r"/>
 </robot>

File: ndo_description/urdf/wheel.urdf.xacro (robot description, xacro)
@@ -1,4 +1,4 @@
 <robot xmlns:xacro="http://www.ros.org/wiki/xacro" name="ndo_wheel">
-    <xacro:macro name="wheel" params="position side spring_stiffness spring_reference">
+    <xacro:macro name="wheel" params="position side">
         <xacro:property name="wheel_radius" value="0.063"/>
         <xacro:property name="wheel_width" value="0.06"/>
@@ -80,21 +80,4 @@
             <axis xyz="0 1 0"/>
         </joint>
-        <!-- Physical properties for the wheels -->
-        <!-- Reference https://www.engineeringtoolbox.com/friction-coefficients-d_778.html -->
-        <gazebo reference="${prefix}_link">
-            <material>Gazebo/FlatBlack</material>
-            <mu1 value="1.0"/>
-            <mu2 value="0.2"/>
-            <kp value="1.0E12"/>
-            <kd value="1.0"/>
-            <fdir1 value="1 0 0"/>
-            <minDepth>0.005</minDepth>
-        </gazebo>
-        <gazebo reference="${prefix}_adptr_joint">
-            <material>Gazebo/DarkYellow</material>
-            <implicitSpringDamper>true</implicitSpringDamper>
-            <springStiffness>${spring_stiffness}</springStiffness>
-            <springReference>${spring_reference}</springReference>
-        </gazebo>
     </xacro:macro>
 </robot>

Commit message: add robot localization

File: ndo_description/urdf/ndo.urdf.xacro (robot description, xacro)
@@ -45,4 +45,21 @@
     <!-- TODO Should probably be dynamic since the robot has a suspension system -->
     <link name="base_footprint"/>
+    <link name="imu_link">
+        <visual>
+            <geometry>
+                <box size="0.01 0.01 0.01"/>
+            </geometry>
+        </visual>
+        <collision>
+            <geometry>
+                <box size="0.01 0.01 0.01"/>
+            </geometry>
+        </collision>
+        <inertial>
+            <origin xyz="0 0 0" rpy="0 0 0"/>
+            <mass value="0.01"/>
+            <inertia ixx="1.6666666666666668e-7" ixy="0.0" ixz="0.0" iyy="1.6666666666666668e-7" iyz="0.0" izz="1.6666666666666668e-7"/>
+        </inertial>
+    </link>
     <!-- Joint base_link with base_footprint to place it at ground level -->
     <joint name="base_joint" type="fixed">
@@ -51,8 +68,13 @@
         <origin xyz="0.0 0.0 ${footprint_zoff}" rpy="0 0 0"/>
     </joint>
-    <joint name="body_link" type="fixed">
+    <joint name="body_joint" type="fixed">
         <parent link="base_link"/>
         <child link="body_link"/>
         <origin xyz="0 0 0" rpy="0 0 0"/>
+    </joint>
+    <joint name="imu_joint" type="fixed">
+        <parent link="base_link"/>
+        <child link="imu_link"/>
+        <origin xyz="0.1 0.04 0.02" rpy="0 0 0"/>
     </joint>
     <!-- Create wheels -->
